File: test_subdir/test_subdir.kicad_pcb (KiCad board)
At the start: 4 copper layers, 49.8 x 48.2 mm, 12 parts, among them J1 Conn_01x08_Male, J2 Conn_01x08_Male, J3 Conn_01x08_Male, J4 USB_B, J5 Conn_01x08_Male, J6 Conn_01x06_Male, U1 FT2232H, Y1 12 MHz

Commit message: Test 6
Parts:
- removed C1, C2: 27 pF, Capacitor_THT:C_Disc_D3.0mm_W1.6mm_P2.50mm
- removed J3, J5: Conn_01x08_Male, Connector_PinHeader_2.54mm:PinHeader_1x08_P2.54mm_Vertical
- removed J4: USB_B, Connector_USB:USB_B_OST_USB-B1HSxx_Horizontal
- removed J6: Conn_01x06_Male, Connector_PinSocket_2.54mm:PinSocket_1x06_P2.54mm_Vertical
- removed R1: 2k2, Resistor_THT:R_Axial_DIN0207_L6.3mm_D2.5mm_P5.08mm_Vertical
- removed R2: 12k 1%, Resistor_THT:R_Axial_DIN0207_L6.3mm_D2.5mm_P5.08mm_Vertical
- removed U1: FT2232H, Package_QFP:LQFP-64_10x10mm_P0.5mm
- removed Y1: 12 MHz, Crystal:Crystal_HC49-U_Vertical
- J1, J2: value Conn_01x08_Male -> Conn_01x04_Pin; footprint Connector_PinHeader_2.54mm:PinHeader_1x08_P2.54mm_Vertical -> Connector_PinSocket_2.54mm:PinSocket_1x04_P2.54mm_Vertical
- moved J1 107.0 mm to (67.8, 67.3)
- moved J2 77.4 mm to (72.4, 67.3), turned to 0 degrees
Connections:
- J1 pad 1: Net-(J1-Pad1) -> Net-(J1-Pin_1)
- J1 pad 2: Net-(J1-Pad2) -> Net-(J1-Pin_2)
- J1 pad 3: Net-(J1-Pad3) -> Net-(J1-Pin_3)
- J1 pad 4: Net-(J1-Pad4) -> Net-(J1-Pin_4)
- J2 pad 1: Net-(J2-Pad1) -> Net-(J1-Pin_1)
- J2 pad 2: Net-(J2-Pad2) -> Net-(J1-Pin_2)
- J2 pad 3: Net-(J2-Pad3) -> Net-(J1-Pin_3)
- J2 pad 4: Net-(J2-Pad4) -> Net-(J1-Pin_4)
Routing:
- net +5V: track 60.0 -> 0.00 mm
- net Net-(J3-Pad7): track 27.0 -> 0.00 mm
- net Net-(U1-Pad12): track 25.9 -> 0.00 mm
- net Net-(J3-Pad8): track 25.4 -> 0.00 mm
- net Net-(J1-Pad1): track 24.0 -> 0.00 mm
- net Net-(J3-Pad6): track 22.3 -> 0.00 mm
- net Net-(J1-Pad2): track 22.1 -> 0.00 mm
- net Net-(J2-Pad8): track 21.1 -> 0.00 mm
- net Net-(J5-Pad1): track 20.9 -> 0.00 mm
- net Net-(J6-Pad1): track 20.8 -> 0.00 mm
- net Net-(J3-Pad5): track 20.6 -> 0.00 mm
- net Net-(J1-Pad3): track 20.6 -> 0.00 mm
- net Net-(J2-Pad7): track 20.3 -> 0.00 mm
- net Net-(J2-Pad1): track 19.9 -> 0.00 mm
- net Net-(J3-Pad4): track 19.8 -> 0.00 mm
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- removed copper zone on In2.Cu, net +3V3
- removed copper zone on GND.Cu, net GND
Other:
- board size 49.8 x 48.2 mm -> 17.8 x 21.6 mm
- copper layers 4 -> 2
- net class Default removed
- rule pad_to_mask_clearance: 0.05 -> 0
