File: test_subdir/test_subdir.kicad_sch (KiCad schematic)
At the start: 12 parts, among them J1 Conn_01x08_Male, J2 Conn_01x08_Male, J3 Conn_01x08_Male, J4 USB_B, J5 Conn_01x08_Male, J6 Conn_01x06_Male, U1 FT2232H, Y1 12 MHz

Commit message: Test 6
Parts:
- removed C1, C2: 27 pF, Capacitor_THT:C_Disc_D3.0mm_W1.6mm_P2.50mm, symbol Device:C
- removed J1, J2, J3, J5: Conn_01x08_Male, Connector_PinHeader_2.54mm:PinHeader_1x08_P2.54mm_Vertical, symbol test_subdir-rescue:Conn_01x08_Male-Connector
- removed J4: USB_B, Connector_USB:USB_B_OST_USB-B1HSxx_Horizontal, symbol test_subdir-rescue:USB_B-Connector
- removed J6: Conn_01x06_Male, Connector_PinSocket_2.54mm:PinSocket_1x06_P2.54mm_Vertical, symbol test_subdir-rescue:Conn_01x06_Male-Connector
- removed R1: 2k2, Resistor_THT:R_Axial_DIN0207_L6.3mm_D2.5mm_P5.08mm_Vertical, symbol Device:R
- removed R2: 12k 1%, Resistor_THT:R_Axial_DIN0207_L6.3mm_D2.5mm_P5.08mm_Vertical, symbol Device:R
- removed U1: FT2232H, Package_QFP:LQFP-64_10x10mm_P0.5mm, symbol test_subdir-rescue:FT2232H-ft
- removed Y1: 12 MHz, Crystal:Crystal_HC49-U_Vertical, symbol Device:Crystal
- added J1, J2: Conn_01x04_Pin, Connector_PinSocket_2.54mm:PinSocket_1x04_P2.54mm_Vertical, symbol Connector:Conn_01x04_Pin
Connections:
- new net: J1.1 (Pin_1), J2.1 (Pin_1)
- new net: J1.2 (Pin_2), J2.2 (Pin_2)
- new net: J1.3 (Pin_3), J2.3 (Pin_3)
- new net: J1.4 (Pin_4), J2.4 (Pin_4)
- no-connect marks 2 -> 0
Other:
- note removed: "Don't try this at home ;-) This is a test schematic, far from real applications."
